Commit message: + move inertial origin to the center of base link. Fix path.

File: urdf/brov2.urdf (robot description, URDF)
Before this commit: robot brov, 7 links, 6 joints
Links:
- link base_link: geometry visual mesh filename=../bluerov_ffg/mesh/BROV2-rdx.stl

Commit message: + inertia for thrusters

File: urdf/brov2.urdf (robot description, URDF)
Before this commit: robot brov, 7 links, 6 joints
Links:
- link thr1: mass None -> 0.1
- link thr2: mass None -> 0.1
- link thr3: mass None -> 0.1
- link thr4: mass None -> 0.1
- link thr5: mass None -> 0.1
- link thr6: mass None -> 0.1

Commit message: + try 6dof thrusters config

File: urdf/brov2.urdf (robot description, URDF)
Before this commit: robot brov, 7 links, 6 joints
Joints:
- joint thr1: origin xyz=0.125 -0.115 -0.07 rpy=0.0 1.57079632679 0.7 -> xyz=0.125 -0.115 0.07 rpy=0.0 1.57079632679 0.7
- joint thr2: origin xyz=0.125 0.115 -0.07 rpy=0.0 1.57079632679 -0.7 -> xyz=0.125 0.115 0.07 rpy=0.0 1.57079632679 -0.7
